File: PCB/UPL_KeyBoard.brd (EAGLE design)
At the start: 320 x 153 mm, 48 parts

Commit message: final design added
Parts:
- flipped J1 to the bottom
Routing:
- net LED_START: track 130.1 -> 62.9 mm, vias 2 -> 4
- net BTN_ROW_4: track 317.9 -> 251.9 mm, vias 9 -> 7
- net BTN_COL_5: track 350.8 -> 409.3 mm
- net LED_OUTPUT: track 62.0 -> 112.6 mm, vias 2 -> 4
- net BTN_ROW_2: track 200.1 -> 156.7 mm, vias 7 -> 5
- net LED_SINGLE: track 68.9 -> 43.6 mm
- net BTN_COL_8: track 285.0 -> 266.6 mm, vias 4 -> 6
- net LED_DATA: track 78.3 -> 60.1 mm
- net BTN_ROW_3: track 199.9 -> 183.9 mm, vias 5 -> 7
- net BTN_ROW_1: track 115.7 -> 131.5 mm, vias 1 -> 2
- net BTN_ROW_5: track 322.6 -> 307.4 mm, vias 2 -> 4
- net BTN_ROW_6: track 320.2 -> 335.3 mm
- net LED_A: track 322.3 -> 334.3 mm
- net BTN_COL_7: track 104.6 -> 114.9 mm
- net BTN_ROW_7: track 395.4 -> 405.6 mm
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Other:
- board text added: "BVKSound UPL Analyzer 20/04/2020"

Commit message: Removed trailing trace, final design, Freeze
Routing:
- net BTN_ROW_3: track 183.9 -> 176.9 mm
Changed lines of the file:
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@@
 <grid distance="0.07" unitdist="mm" unit="mm" style="lines" multiple="1" display="yes" altdistance="0.1" altunitdist="mm" altunit="mm"/>
 <layers>
-<layer number="1" name="Top" color="4" fill="1" visible="no" active="yes"/>
+<layer number="1" name="Top" color="4" fill="1" visible="yes" active="yes"/>
 <layer number="2" name="Route2" color="1" fill="3" visible="no" active="no"/>
 <layer number="3" name="Route3" color="4" fill="3" visible="no" active="no"/>
@@
 <wire x1="299.1" y1="124.9" x2="299.1" y2="138" width="0.5" layer="1"/>
 <wire x1="299.1" y1="138" x2="299.03" y2="138" width="0.5" layer="1"/>
-<wire x1="240.96" y1="92.98" x2="234" y2="92.98" width="0.5" layer="1"/>
 <wire x1="261.28" y1="128.18" x2="261.28" y2="119.7" width="0.5" layer="1"/>
 <wire x1="261.28" y1="119.7" x2="261.2" y2="119.7" width="0.5" layer="1"/>
