File: KEYBOARD/PCB/SMD Buttons/UPL_KeyBoard.sch (KiCad schematic (older format))
At the start: 48 parts, among them J1 Conn_02x13_Odd_Even, SW1 START, SW10 8, SW11 9, SW12 SELECT, SW13 HELP, SW14 TABRIGHT, SW15 4, SW16 5, SW17 6, SW18 BACKSP, SW19 TABLEFT, SW2 SINGLE, SW20 PGUP, SW21 1, SW22 2, SW23 3, SW24 CANCEL, SW25 PGDOWN, SW26 0, SW27 POINT, SW28 MINUS, SW29 ENTER, SW3 STOP, SW30 LEFT, SW31 RIGHT, SW32 UP, SW33 DOWN, SW34 F1, SW35 F2, SW36 F3, SW37 F4, SW38 F5, SW39 F6, SW4 HCOPY, SW40 F7, SW41 F8, SW5 SYSTEM, SW6 CONTRAST, SW7 OUTPUT, SW8 LOCAL, SW9 7

Commit message: Finalized design with FFC Connector
Parts:
- J1: footprint Connector_PinHeader_2.54mm:PinHeader_2x13_P2.54mm_Vertical -> BVKSound:0520443445_Mirrored
Changed lines of the file:
@@
 F 0 "J1" H 3200 2917 50  0000 C CNN
 F 1 "Conn_02x13_Odd_Even" H 3200 2826 50  0000 C CNN
-F 2 "Connector_PinHeader_2.54mm:PinHeader_2x13_P2.54mm_Vertical" H 3150 2100 50  0001 C CNN
+F 2 "BVKSound:0520443445_Mirrored" H 3150 2100 50  0001 C CNN
 F 3 "~" H 3150 2100 50  0001 C CNN
 	1    3150 2100
